File: TMP102_Temperature_Sensor.kicad_pcb (KiCad board)
At the start: 2 copper layers, 30.2 x 30.2 mm, 15 parts, among them J1 JST_SH_SM06B-SRSS-TB_1x06-1MP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, J4 Conn_01x04, U1 M24C02-FMN, U2 TMP102xxDRL

Commit message: Change to 10K pullup resistor on interrupt line.
Parts:
- R1: value 100K -> 10K
Changed lines of the file:
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@@
 			)
 		)
-		(property "Value" "100K"
+		(property "Value" "10K"
 			(at 0 1.43 90)
 			(layer "F.Fab")
@@
 			)
 		)
-		(property "MPN" ""
+		(property "MPN" "C25804"
 			(at 0 0 270)
 			(unlocked yes)
@@
 			)
 		)
-		(property "Feeder" ""
+		(property "Feeder" "8mm"
 			(at 0 0 270)
 			(unlocked yes)
